File: src/pcb/IoT MD2 2019-2020/electrical_scheme.sch (EAGLE design)
At the start: 17 parts, among them P1 S2B-PH-SM4-TB, Q1 32.768kHz, U1 ATSAMD21E18A-AF, U2 TPS73533DRVT

Commit message: Changed electrical scheme + image
Parts:
- removed C4: 0.1uF, capacitor-wima:C2.5/5
- removed C5: 1uF, rcl:CPOL-EUE5-5
- removed U2: TPS73533DRVT, TPS73533DRVT:TPS73533DRVT
- added C6: 15pF, rcl:C-EUC1608
- C1: device capacitor-wima:C2.5/5 -> rcl:C-EUC1608
- C2: value 1uF -> 470pF; device capacitor-wima:C2.5/5 -> rcl:C-EUC1608
- C3: value 0.01uF -> 15pF; device capacitor-wima:C2.5/5 -> rcl:C-EUC1608
- C7: value 15pF -> 0.1uF; device capacitor-wima:C2.5/5 -> rcl:C-EUC1608
- C8: value 15pF -> 1uF; device capacitor-wima:C2.5/5 -> rcl:CPOL-EUC/6032-28R
Connections:
- removed net N$1: C5.+, U1.VDDCORE
- new net VDDCORE: C8.+, U1.VDDCORE
- net 0: now also C2.2, C6.2, C7.2, C8.-, IC1.GND; no longer C2.1, C4.2, C5.-, C7.1, C8.1, U2.GND
- net N$2: now also IC1.EN, IC1.IN; no longer C2.2, U2.EN, U2.IN
- net N$3: now also C2.1, IC1.BYP; no longer C3.1, U2.NR/FB
- net N$4: now also C3.1; no longer C7.2
- net N$5: now also C6.1; no longer C8.2
- net VDD: now also C7.1, IC1.OUT; no longer C4.1, U2.OUT
Other:
- note added: "Load Capacitors MCU"
- moved on the sheet: C1, C2, C3, C7, IC1, P1, Q1

Commit message: Added board, modified scheme grounds for ground plane
Connections:
- net 0 renamed GND
- removed net SWCLK: U1.PA30
- net MISO: now also SV2.4; no longer SV2.7
- net MOSI: now also SV2.7; no longer SV2.6
- net N$4: now also Q1.1; no longer Q1.2
- net N$5: now also Q1.2; no longer Q1.1
- net NSS: now also SV2.5; no longer SV2.4
- net RESET_LORA: now also U1.PA15; no longer U1.PA24
- net SCK: now also SV2.6; no longer SV2.5
- net SWDCLK: now also U1.PA30
Other:
- moved on the sheet: Q1

Commit message: Deleted board + added reset circuit into scheme -> TODO: add smd switch into reset circuit
Parts:
- added C4: 100nF, rcl:C-EUC1608
- added JP1: (no value), pinhead:PINHD-1X2
- added R1: 10k, rcl:R-EU_R0805
Connections:
- net GND: now also C4.2, JP1.2
- net RESET: now also C4.1, JP1.1, R1.1
- net VDD: now also R1.2
Other:
- note added: "RESET Scheme"
- moved on the sheet: C1, C2, IC1, P1

Commit message: Board scheme
Connections:
- removed net N$3: C2.1, IC1.BYP
- new net N$1: C2.2, IC1.BYP
- net GND: now also C1.1, C2.1, SV5.4; no longer C1.2, C2.2, SV5.3
- net SCL: now also SV3.1, SV4.1; no longer SV3.2, SV4.2
- net SDA: now also SV3.2, SV4.2; no longer SV3.1, SV4.1
- net VDD: now also C1.2, SV5.3; no longer C1.1, SV5.4
Other:
- moved on the sheet: C1, C2
Changed lines of the file:
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@@
 <attribute name="VALUE" x="116.84" y="116.84" size="1.778" layer="96"/>
 </instance>
-<instance part="C1" gate="G$1" x="127" y="121.92" smashed="yes">
-<attribute name="NAME" x="128.524" y="122.301" size="1.778" layer="95"/>
-<attribute name="VALUE" x="128.524" y="117.221" size="1.778" layer="96"/>
-</instance>
-<instance part="C2" gate="G$1" x="91.44" y="114.3" smashed="yes">
-<attribute name="NAME" x="92.964" y="114.681" size="1.778" layer="95"/>
-<attribute name="VALUE" x="92.964" y="109.601" size="1.778" layer="96"/>
+<instance part="C1" gate="G$1" x="127" y="116.84" smashed="yes" rot="R180">
+<attribute name="NAME" x="125.476" y="116.459" size="1.778" layer="95" rot="R180"/>
+<attribute name="VALUE" x="125.476" y="121.539" size="1.778" layer="96" rot="R180"/>
+</instance>
+<instance part="C2" gate="G$1" x="91.44" y="111.76" smashed="yes" rot="R180">
+<attribute name="NAME" x="89.916" y="111.379" size="1.778" layer="95" rot="R180"/>
+<attribute name="VALUE" x="89.916" y="116.459" size="1.778" layer="96" rot="R180"/>
 </instance>
 <instance part="C3" gate="G$1" x="185.42" y="73.66" smashed="yes">
@@
 <attribute name="VALUE" x="208.28" y="-15.24" size="1.778" layer="96"/>
 </instance>
-<instance part="GND5" gate="1" x="210.82" y="20.32" smashed="yes">
-<attribute name="VALUE" x="208.28" y="17.78" size="1.778" layer="96"/>
+<instance part="GND5" gate="1" x="210.82" y="22.86" smashed="yes">
+<attribute name="VALUE" x="208.28" y="20.32" size="1.778" layer="96"/>
 </instance>
 <instance part="GND6" gate="1" x="185.42" y="60.96" smashed="yes">
@@
 <net name="VDD" class="0">
 <segment>
-<wire x1="127" y1="129.54" x2="127" y2="124.46" width="0.1524" layer="91"/>
-<wire x1="127" y1="129.54" x2="142.24" y2="129.54" width="0.1524" layer="91"/>
-<junction x="127" y="129.54"/>
+<wire x1="116.84" y1="129.54" x2="127" y2="129.54" width="0.1524" layer="91"/>
 <label x="142.24" y="129.54" size="1.778" layer="95"/>
 <pinref part="IC1" gate="G1" pin="OUT"/>
-<wire x1="116.84" y1="129.54" x2="127" y2="129.54" width="0.1524" layer="91"/>
-<pinref part="C1" gate="G$1" pin="1"/>
+<pinref part="C1" gate="G$1" pin="2"/>
+<wire x1="127" y1="129.54" x2="142.24" y2="129.54" width="0.1524" layer="91"/>
+<wire x1="127" y1="121.92" x2="127" y2="129.54" width="0.1524" layer="91"/>
+<junction x="127" y="129.54"/>
 </segment>
 <segment>
@@
 </segment>
 <segment>
-<wire x1="198.12" y1="27.94" x2="203.2" y2="27.94" width="0.1524" layer="91"/>
-<label x="203.2" y="27.94" size="1.4224" layer="95"/>
-<pinref part="SV5" gate="1" pin="4"/>
-</segment>
-<segment>
 <pinref part="C7" gate="G$1" pin="1"/>
 <wire x1="182.88" y1="124.46" x2="182.88" y2="129.54" width="0.1524" layer="91"/>
@@
 <wire x1="83.82" y1="81.28" x2="83.82" y2="88.9" width="0.1524" layer="91"/>
 <label x="83.82" y="88.9" size="1.778" layer="95"/>
+</segment>
+<segment>
+<pinref part="SV5" gate="1" pin="3"/>
+<wire x1="198.12" y1="25.4" x2="203.2" y2="25.4" width="0.1524" layer="91"/>
+<label x="203.2" y="25.4" size="1.4224" layer="95"/>
 </segment>
 </net>
@@
 <net name="SCL" class="0">
 <segment>
+<pinref part="U1" gate="G$1" pin="PA23"/>
+<wire x1="259.08" y1="73.66" x2="266.7" y2="73.66" width="0.1524" layer="91"/>
+<label x="266.7" y="73.66" size="1.9304" layer="95"/>
+</segment>
+<segment>
+<pinref part="SV4" gate="1" pin="1"/>
+<wire x1="198.12" y1="-12.7" x2="203.2" y2="-12.7" width="0.1524" layer="91"/>
+<label x="203.2" y="-12.7" size="1.4224" layer="95"/>
+</segment>
+<segment>
+<pinref part="SV3" gate="1" pin="1"/>
+<wire x1="152.4" y1="-12.7" x2="157.48" y2="-12.7" width="0.1524" layer="91"/>
+<label x="157.48" y="-12.7" size="1.4224" layer="95"/>
+</segment>
+</net>
+<net name="SDA" class="0">
+<segment>
+<pinref part="U1" gate="G$1" pin="PA22"/>
+<wire x1="259.08" y1="76.2" x2="266.7" y2="76.2" width="0.1524" layer="91"/>
+<label x="266.7" y="76.2" size="1.9304" layer="95"/>
+</segment>
+<segment>
+<pinref part="SV4" gate="1" pin="2"/>
+<wire x1="198.12" y1="-10.16" x2="203.2" y2="-10.16" width="0.1524" layer="91"/>
+<label x="203.2" y="-10.16" size="1.4224" layer="95"/>
+</segment>
+<segment>
 <pinref part="SV3" gate="1" pin="2"/>
 <wire x1="152.4" y1="-10.16" x2="157.48" y2="-10.16" width="0.1524" layer="91"/>
 <label x="157.48" y="-10.16" size="1.4224" layer="95"/>
 </segment>
-<segment>
-<pinref part="SV4" gate="1" pin="2"/>
-<wire x1="198.12" y1="-10.16" x2="203.2" y2="-10.16" width="0.1524" layer="91"/>
-<label x="203.2" y="-10.16" size="1.4224" layer="95"/>
-</segment>
-<segment>
-<pinref part="U1" gate="G$1" pin="PA23"/>
-<wire x1="259.08" y1="73.66" x2="266.7" y2="73.66" width="0.1524" layer="91"/>
-<label x="266.7" y="73.66" size="1.9304" layer="95"/>
-</segment>
-</net>
-<net name="SDA" class="0">
-<segment>
-<pinref part="SV3" gate="1" pin="1"/>
-<wire x1="152.4" y1="-12.7" x2="157.48" y2="-12.7" width="0.1524" layer="91"/>
-<label x="157.48" y="-12.7" size="1.4224" layer="95"/>
-</segment>
-<segment>
-<pinref part="SV4" gate="1" pin="1"/>
-<wire x1="198.12" y1="-12.7" x2="203.2" y2="-12.7" width="0.1524" layer="91"/>
-<label x="203.2" y="-12.7" size="1.4224" layer="95"/>
-</segment>
-<segment>
-<pinref part="U1" gate="G$1" pin="PA22"/>
-<wire x1="259.08" y1="76.2" x2="266.7" y2="76.2" width="0.1524" layer="91"/>
-<label x="266.7" y="76.2" size="1.9304" layer="95"/>
-</segment>
 </net>
 <net name="RX" class="0">
@@
 <wire x1="259.08" y1="88.9" x2="266.7" y2="88.9" width="0.1524" layer="91"/>
 <label x="266.7" y="88.9" size="1.778" layer="95"/>
-</segment>
-</net>
-<net name="N$3" class="0">
-<segment>
-<pinref part="IC1" gate="G1" pin="BYP"/>
-<wire x1="96.52" y1="119.38" x2="91.44" y2="119.38" width="0.1524" layer="91"/>
-<pinref part="C2" gate="G$1" pin="1"/>
-<wire x1="91.44" y1="119.38" x2="91.44" y2="116.84" width="0.1524" layer="91"/>
 </segment>
 </net>
@@
 </segment>
 <segment>
-<wire x1="198.12" y1="25.4" x2="210.82" y2="25.4" width="0.1524" layer="91"/>
-<wire x1="210.82" y1="25.4" x2="210.82" y2="22.86" width="0.1524" layer="91"/>
-<pinref part="SV5" gate="1" pin="3"/>
-<pinref part="GND5" gate="1" pin="GND"/>
-</segment>
-<segment>
 <pinref part="C6" gate="G$1" pin="2"/>
 <wire x1="195.58" y1="68.58" x2="195.58" y2="66.04" width="0.1524" layer="91"/>
@@
 <wire x1="109.22" y1="106.68" x2="109.22" y2="104.14" width="0.1524" layer="91"/>
 <junction x="109.22" y="106.68"/>
-<pinref part="C1" gate="G$1" pin="2"/>
-<wire x1="127" y1="116.84" x2="127" y2="106.68" width="0.1524" layer="91"/>
 <wire x1="127" y1="106.68" x2="109.22" y2="106.68" width="0.1524" layer="91"/>
 <pinref part="P1" gate="G$1" pin="2"/>
 <wire x1="81.28" y1="106.68" x2="81.28" y2="125.73" width="0.1524" layer="91"/>
 <wire x1="109.22" y1="106.68" x2="91.44" y2="106.68" width="0.1524" layer="91"/>
-<pinref part="C2" gate="G$1" pin="2"/>
+<pinref part="GND7" gate="1" pin="GND"/>
+<pinref part="C2" gate="G$1" pin="1"/>
 <wire x1="91.44" y1="106.68" x2="81.28" y2="106.68" width="0.1524" layer="91"/>
 <wire x1="91.44" y1="109.22" x2="91.44" y2="106.68" width="0.1524" layer="91"/>
 <junction x="91.44" y="106.68"/>
-<pinref part="GND7" gate="1" pin="GND"/>
+<pinref part="C1" gate="G$1" pin="1"/>
+<wire x1="127" y1="114.3" x2="127" y2="106.68" width="0.1524" layer="91"/>
 </segment>
 <segment>
@@
 <wire x1="114.3" y1="53.34" x2="114.3" y2="50.8" width="0.1524" layer="91"/>
 </segment>
-</net>
+<segment>
+<pinref part="SV5" gate="1" pin="4"/>
+<pinref part="GND5" gate="1" pin="GND"/>
+<wire x1="198.12" y1="27.94" x2="210.82" y2="27.94" width="0.1524" layer="91"/>
+<wire x1="210.82" y1="27.94" x2="210.82" y2="25.4" width="0.1524" layer="91"/>
+</segment>
+</net>
+<net name="N$1" class="0">
+<segment>
+<pinref part="IC1" gate="G1" pin="BYP"/>
+<wire x1="96.52" y1="119.38" x2="91.44" y2="119.38" width="0.1524" layer="91"/>
+<pinref part="C2" gate="G$1" pin="2"/>
+<wire x1="91.44" y1="119.38" x2="91.44" y2="116.84" width="0.1524" layer="91"/>
+</segment>
+</net>
