File: src/pcb/IoT MD2 2019-2020/mcu_module.sch (EAGLE design)
At the start: 17 parts, among them Q1 32.768kHz, U1 ATSAMD21E18A-AF

Commit message: Finished PCB, added gerber files
Parts:
- added C7: 1uF, rcl:C-EUC0805
- added R2: 330, rcl:R-EU_R0805
- added S1: (no value), switch-omron:10-XX
Connections:
- new net N$3: R2.1, S1.S
- net GND: now also C7.2, S1.P
- net MISO: now also JP4.1; no longer JP4.2
- net MOSI: now also JP4.4; no longer JP4.5
- net NSS: now also JP4.2; no longer JP4.3
- net RESET: now also R2.2
- net RESET_LORA: now also JP4.5, U1.PA15; no longer JP4.1, U1.PA24
- net SCK: now also JP4.3; no longer JP4.4
- net SCL: now also U1.PA22; no longer U1.PA23
- net SDA: now also U1.PA23; no longer U1.PA22
- net VDDCORE: now also C7.1
Other:
- note added: "MCU"
- note added: "Polarized"
- moved on the sheet: C6, R1
