File: src/pcb/IoT MD2 2019-2020/mcu_module.sch (EAGLE design)
At the start: 20 parts, among them IC2 ATSAMD21G18A-AU, Y1 ABS07-32.768KHZ-T

Commit message: Gerber files MCU v2, IMAGES MCU V2 added
Parts:
- renumbered JP1 to SWD_DEBUGGER, JP2 to INPUT, JP3 to RESET, JP5 to GPS, JP6 to HUMIDITY, JP7 to 9DOF, JP8 to LORA
Connections:
- removed net VDDIN: IC2.VDDIN
- net DIO0: now also LORA.9; no longer LORA.5
- net DIO2: now also LORA.5; no longer LORA.9
- net GND: now also 9DOF.1, HUMIDITY.1, IC2.GND_3; no longer 9DOF.2, HUMIDITY.2
- net MISO: now also LORA.6; no longer LORA.1
- net MOSI: now also LORA.1; no longer LORA.4
- net NSS: now also LORA.4; no longer LORA.3
- net RESET_LORA: now also LORA.3; no longer LORA.6
- net VDD: now also 9DOF.2, HUMIDITY.2, IC2.VDDIN, IC2.VDDIO_2; no longer 9DOF.1, HUMIDITY.1
Other:
- moved on the sheet: C5, C7
