File: src/pcb/IoT MD2 2019-2020/mcu_module.brd (EAGLE design)
At the start: 64.8 x 54.3 mm, 20 parts, among them Q1 32.768kHz, U1 ATSAMD21E18A-AF

Commit message: Optimized pcb design
Parts:
- moved JP7 16.5 mm to (69.8, 21.6)
- moved JP5 15.2 mm to (47.0, 21.6)
- moved IC1 14.2 mm to (73.7, 41.9)
- moved JP2 14.2 mm to (73.7, 49.5)
- moved C3 14.2 mm to (71.1, 31.8)
- moved C4 14.2 mm to (71.1, 36.8)
- moved JP6 14.0 mm to (64.8, 21.6)
- moved JP4 12.7 mm to (58.4, 25.4)
- moved JP1 6.35 mm to (43.2, 52.1), turned to 0 degrees
- moved JP3 3.59 mm to (53.3, 53.3)
Routing:
- net GND: track 285.7 -> 209.1 mm
- net VDD: track 148.0 -> 105.0 mm
- net RESET: track 53.6 -> 31.9 mm
- net SDA: track 47.5 -> 31.0 mm
- net SCL: track 48.6 -> 32.0 mm
- net RX: track 23.0 -> 7.75 mm
- net TX: track 20.1 -> 4.88 mm
- net MISO: track 21.4 -> 8.69 mm
- net SCK: track 22.5 -> 9.80 mm
- net NSS: track 21.8 -> 9.08 mm
- net MOSI: track 23.2 -> 10.5 mm
- net RESET_LORA: track 26.5 -> 14.5 mm
- net SWDIO: track 19.2 -> 24.0 mm
- net SWDCLK: track 22.3 -> 24.8 mm
Other:
- board size 64.8 x 54.3 mm -> 47 x 44.1 mm
