File: src/pcb/IoT MD2 2019-2020/mcu_module.brd (EAGLE design)
At the start: 47 x 44.1 mm, 20 parts, among them IC2 ATSAMD21G18A-AU, Y1 ABS07-32.768KHZ-T

Commit message: Gerber files MCU v2, IMAGES MCU V2 added
Parts:
- removed JP1, JP8: (no value), pinhead:2X05
- removed JP2, JP3: (no value), pinhead:1X02
- removed JP5, JP6, JP7: (no value), pinhead:1X04
- added 9DOF, GPS, HUMIDITY: (no value), pinhead:1X04
- added INPUT, RESET: (no value), pinhead:1X02
- added LORA, SWD_DEBUGGER: (no value), pinhead:2X05
- moved IC2 68.5 mm to (81.3, 53.3)
- moved Y1 59.5 mm to (72.4, 55.9), turned to 270 degrees
- moved C5 48.3 mm to (83.8, 64.8)
- moved C6 48.0 mm to (87.6, 71.1), turned to 90 degrees
- moved C7 41.6 mm to (80.0, 64.8), turned to 90 degrees
- moved C2 41.1 mm to (68.8, 54.0)
- moved S1 39.8 mm to (80.0, 80.0), turned to 180 degrees
- moved R1 39.7 mm to (80.0, 71.1), turned to 180 degrees
- moved R2 38.7 mm to (83.8, 71.1), turned to 270 degrees
- moved C1 36.4 mm to (66.0, 55.9), turned to 270 degrees
- moved C3 22.2 mm to (62.2, 52.1), turned to 0 degrees
- moved IC1 14.2 mm to (61.0, 48.3), turned to 270 degrees
- moved C4 10.8 mm to (63.5, 44.5), turned to 0 degrees
Connections:
- removed net N$10: IC2.30
- removed net N$4: IC2.24
- removed net N$5: IC2.25
- removed net N$6: IC2.26
- removed net N$7: IC2.27
- removed net N$8: IC2.28
- removed net N$9: IC2.29
- removed net VDDIN: IC2.44
- net DIO0: now also IC2.21, LORA.9; no longer JP8.5
- net DIO1: now also IC2.22, LORA.7; no longer JP8.7
- net DIO2: now also IC2.23, LORA.5; no longer JP8.9
- net GND: now also 9DOF.1, GPS.3, HUMIDITY.1, IC2.42, INPUT.2, LORA.8, RESET.2, SWD_DEBUGGER.3, SWD_DEBUGGER.5; no longer JP1.3, JP1.5, JP2.2, JP3.2, JP5.3, JP6.2, JP7.2, JP8.8
- net INPUT: now also INPUT.1; no longer JP2.1
- net MISO: now also IC2.28, LORA.6; no longer JP8.1
- net MOSI: now also IC2.25, LORA.1; no longer JP8.4
- net NSS: now also IC2.27, LORA.4; no longer JP8.3
- net RESET: now also RESET.1, SWD_DEBUGGER.10; no longer JP1.10, JP3.1
- net RESET_LORA: now also IC2.24, LORA.3; no longer JP8.6
- net RX: now also GPS.2; no longer JP5.2
- net SCK: now also IC2.26, LORA.2; no longer JP8.2
- net SCL: now also 9DOF.3, HUMIDITY.3; no longer JP6.3, JP7.3
- net SDA: now also 9DOF.4, HUMIDITY.4; no longer JP6.4, JP7.4
- net SWDCLK: now also SWD_DEBUGGER.4; no longer JP1.4
- net SWDIO: now also SWD_DEBUGGER.2; no longer JP1.2
- net TX: now also GPS.1; no longer JP5.1
- net VDD: now also 9DOF.2, GPS.4, HUMIDITY.2, IC2.36, IC2.44, LORA.10, SWD_DEBUGGER.1; no longer JP1.1, JP5.4, JP6.1, JP7.1, JP8.10
Routing:
- net GND: track 171.1 -> 208.7 mm
- net VDD: track 67.3 -> 104.1 mm
- net MISO: track 0.00 -> 19.0 mm
- net SDA: track 28.9 -> 12.0 mm
- net SCL: track 29.5 -> 12.8 mm
- net DIO0: track 0.00 -> 16.6 mm
- net NSS: track 0.00 -> 15.5 mm
- net RESET_LORA: track 0.00 -> 14.2 mm
- net DIO1: track 0.00 -> 13.9 mm
- net DIO2: track 0.00 -> 12.9 mm
- net SCK: track 0.00 -> 11.0 mm
- net RESET: track 29.0 -> 39.9 mm
- net N$1: track 1.90 -> 11.6 mm
- net SWDCLK: track 24.5 -> 15.1 mm
- net MOSI: track 0.00 -> 7.81 mm
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Other:
- board size 47 x 44.1 mm -> 44.4 x 47.9 mm
