File: src/pcb/IoT MD2 2019-2020/lora_module.sch (EAGLE design)
At the start: 4 parts, among them J1 U.FL-R-SMT-1(10)

Commit message: Gerber files
Parts:
- added C1: 1uF, rcl:C-EUC0805
- added C2: 10uF, rcl:C-EUC0805
- added C3: 100nF, rcl:C-EUC0805
Connections:
- net DIO0: now also SV2.3; no longer SV2.1
- net DIO1: now also SV2.4; no longer SV2.2
- net DIO2: now also SV2.5; no longer SV2.3
- net GND: now also C1.2, C2.2, C3.2, SV2.1; no longer SV1.2
- net MISO: now also SV1.5; no longer SV1.3
- net MOSI: now also SV1.4; no longer SV2.5
- net NSS: now also SV1.2; no longer SV1.4
- net RESET_LORA: now also SV1.1; no longer SV2.4
- net SCK: now also SV1.3; no longer SV1.5
- net VDD: now also C1.1, C2.1, C3.1, SV2.2; no longer SV1.1
