File: src/pcb/IoT MD2 2019-2020/lora_module.brd (EAGLE design)
At the start: 27.9 x 32.7 mm, 7 parts, among them J1 U.FL-R-SMT-1(10)

Commit message: Updated gerber files
Other:
- board size 27.9 x 32.7 mm -> 25.4 x 31.4 mm
Changed lines of the file:
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@@
 <drawing>
 <settings>
-<setting alwaysvectorfont="yes"/>
+<setting alwaysvectorfont="no"/>
 <setting verticaltext="up"/>
 </settings>
@@
 <fusionsync huburn="a.YnVzaW5lc3M6c3R1ZGVudDEwMzky" projecturn="a.YnVzaW5lc3M6c3R1ZGVudDEwMzkyI0QyMDE5MTAxMTIyNTQ4NzIwNg" f3durn="urn:adsk.wipprod:dm.lineage:o5PwCKtQTq-g7Tc5t2Tl6A" pcbguid="f2edb4a1-dce4-4dac-8719-28d8a49f27ce" lastpulledtime="" lastsyncedchangeguid="c10cce32-c4fd-c831-0186-31674836a32d"/>
 <plain>
-<wire x1="0" y1="38.1" x2="27.92" y2="38.1" width="0" layer="20"/>
-<wire x1="27.92" y1="38.1" x2="27.92" y2="70.79" width="0" layer="20"/>
-<wire x1="27.92" y1="70.79" x2="0" y2="70.79" width="0" layer="20"/>
-<wire x1="0" y1="70.79" x2="0" y2="38.1" width="0" layer="20"/>
+<wire x1="1.27" y1="38.1" x2="26.65" y2="38.1" width="0" layer="20"/>
+<wire x1="26.65" y1="38.1" x2="26.65" y2="69.52" width="0" layer="20"/>
+<wire x1="26.65" y1="69.52" x2="1.27" y2="69.52" width="0" layer="20"/>
+<wire x1="1.27" y1="69.52" x2="1.27" y2="38.1" width="0" layer="20"/>
 </plain>
 <attributes>
@@
 <wire x1="25.08" y1="40.32" x2="25.08" y2="41.91" width="0.3048" layer="1"/>
 <polygon width="0.3048" layer="1">
-<vertex x="0" y="71.12"/>
-<vertex x="0" y="36.83"/>
-<vertex x="29.21" y="36.83"/>
-<vertex x="29.21" y="71.12"/>
+<vertex x="1.27" y="69.85"/>
+<vertex x="1.27" y="38.1"/>
+<vertex x="26.67" y="38.1"/>
+<vertex x="26.67" y="69.85"/>
 </polygon>
 </signal>
