File: src/pcb/Humidity_sensor/schema/humidity_sensor.brd (EAGLE design)
At the start: 21.3 x 20.3 mm, 6 parts

Commit message: Updated text for pcb
Parts:
- moved SV1 1.27 mm to (3.81, 69.8)
- renumbered U$1 to HUMIDITY
Routing:
- net SCL: track 17.0 -> 19.7 mm
- net GND: track 17.0 -> 19.0 mm
- net VDD: track 42.3 -> 43.8 mm
- net SDA: track 12.1 -> 13.4 mm
Other:
- board size 21.3 x 20.3 mm -> 21.3 x 19.7 mm
- board text added: "GND"
- board text added: "SCL"
- board text added: "SDA"
- board text added: "VDD"
