File: src/pcb/GPS_module/schema/GPS_Module.brd (EAGLE design)
At the start: 23.8 x 25.4 mm, 9 parts, among them J2 U.FL-R-SMT(01), U1 SL876Q5A001T001000

Commit message: Merge conflict fix
Other:
- board size 23.8 x 25.4 mm -> 23.8 x 27.9 mm
Changed lines of the file:
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@@
 </layers>
 <board>
-<fusionsync huburn="a.YnVzaW5lc3M6c3R1ZGVudDk3MjU" projecturn="a.YnVzaW5lc3M6c3R1ZGVudDk3MjUjRDIwMTkxMDA0MjIyNzk2ODA2" f3durn="urn:adsk.wipprod:dm.lineage:NpaNXs29SPKqhJ0U-8d7cw" pcbguid="de09cc18-a3d4-48f8-913a-f04e929a34a4" lastpulledtime="" lastsyncedchangeguid="45d9a472-997a-c3df-27ff-b88bcedcdcec"/>
+<fusionsync huburn="a.YnVzaW5lc3M6c3R1ZGVudDk3MjU" projecturn="a.YnVzaW5lc3M6c3R1ZGVudDk3MjUjRDIwMTkxMDA0MjIyNzk2ODA2" f3durn="urn:adsk.wipprod:dm.lineage:NpaNXs29SPKqhJ0U-8d7cw" pcbguid="de09cc18-a3d4-48f8-913a-f04e929a34a4" lastpulledtime="" lastsyncedchangeguid="ae47f3d3-d591-f2fe-bc63-d4625d2e3dec"/>
 <plain>
-<wire x1="3.81" y1="10.16" x2="20.32" y2="10.16" width="0" layer="20"/>
-<wire x1="20.32" y1="10.16" x2="23.8" y2="13.64" width="0" layer="20"/>
-<wire x1="23.8" y1="13.64" x2="23.8" y2="35.549996875" width="0" layer="20"/>
-<wire x1="23.8" y1="35.549996875" x2="0" y2="35.539840625" width="0" layer="20"/>
-<wire x1="0" y1="35.539840625" x2="0" y2="13.97" width="0" layer="20"/>
-<wire x1="0" y1="13.97" x2="3.81" y2="10.16" width="0" layer="20"/>
+<wire x1="0" y1="39.349840625" x2="0" y2="11.43" width="0" layer="20"/>
+<wire x1="0" y1="11.43" x2="23.8" y2="11.43" width="0" layer="20"/>
+<wire x1="23.8" y1="11.43" x2="23.8" y2="39.359996875" width="0" layer="20"/>
+<wire x1="23.8" y1="39.359996875" x2="0" y2="39.349840625" width="0" layer="20"/>
+<hole x="2.54" y="13.97" drill="3"/>
+<hole x="21.59" y="13.97" drill="3"/>
+<hole x="2.54" y="36.83" drill="3"/>
+<hole x="21.59" y="36.83" drill="3"/>
 </plain>
 <attributes>
@@
 <wire x1="7" y1="25.42" x2="7.3" y2="25.72" width="0.3048" layer="1"/>
 <polygon width="0.1524" layer="1">
-<vertex x="0" y="35.56"/>
-<vertex x="24.13" y="35.56"/>
-<vertex x="24.13" y="13.97"/>
-<vertex x="20.32" y="10.16"/>
-<vertex x="3.81" y="10.16"/>
-<vertex x="0" y="13.97"/>
+<vertex x="0" y="39.37"/>
+<vertex x="24.13" y="39.37"/>
+<vertex x="24.13" y="11.43"/>
+<vertex x="0" y="11.43"/>
 </polygon>
 <contactref element="J2" pad="2"/>
@@
 <wire x1="13.97" y1="25.72" x2="12.38" y2="25.72" width="0.3048" layer="1"/>
 <wire x1="12.38" y1="25.72" x2="11.43" y2="26.67" width="0.3048" layer="1"/>
+<wire x1="18.845" y1="31.75" x2="21.795" y2="31.75" width="0" layer="19" extent="1-1"/>
+<wire x1="11.43" y1="28.26" x2="13.97" y2="32.7" width="0" layer="19" extent="1-1"/>
+<wire x1="7" y1="16.58" x2="7" y2="22.18" width="0" layer="19" extent="1-1"/>
+<wire x1="7" y1="13.38" x2="7" y2="16.58" width="0" layer="19" extent="1-1"/>
+<wire x1="18.4" y1="22.18" x2="13.97" y2="25.72" width="0" layer="19" extent="1-1"/>
+<wire x1="18.4" y1="20.58" x2="18.4" y2="22.18" width="0" layer="19" extent="1-1"/>
+<wire x1="18.4" y1="16.58" x2="18.4" y2="20.58" width="0" layer="19" extent="1-1"/>
+<wire x1="18.4" y1="14.98" x2="18.4" y2="16.58" width="0" layer="19" extent="1-1"/>
+<wire x1="18.4" y1="14.18" x2="18.4" y2="14.98" width="0" layer="19" extent="1-1"/>
 </signal>
 <signal name="VDD">

Commit message: updated shematic of GPS and Humidity
Parts:
- added R3: 1000, rcl:R0402
- R1: value 100 -> 220; device rcl:R0805 -> rcl:R0402
- R2: value 120 -> 330; device rcl:R0805 -> rcl:R0402
Connections:
- net GND: now also R3.1
- net VIN: now also R3.2
Routing:
- net VIN: track 32.7 -> 37.3 mm
- net GND: track 25.2 -> 23.0 mm
Changed lines of the file:
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@@
 </layers>
 <board>
-<fusionsync huburn="a.YnVzaW5lc3M6c3R1ZGVudDk3MjU" projecturn="a.YnVzaW5lc3M6c3R1ZGVudDk3MjUjRDIwMTkxMDA0MjIyNzk2ODA2" f3durn="urn:adsk.wipprod:dm.lineage:NpaNXs29SPKqhJ0U-8d7cw" pcbguid="de09cc18-a3d4-48f8-913a-f04e929a34a4" lastpulledtime="" lastsyncedchangeguid="ae47f3d3-d591-f2fe-bc63-d4625d2e3dec"/>
+<fusionsync huburn="a.YnVzaW5lc3M6c3R1ZGVudDk3MjU" projecturn="a.YnVzaW5lc3M6c3R1ZGVudDk3MjUjRDIwMTkxMDA0MjIyNzk2ODA2" f3durn="urn:adsk.wipprod:dm.lineage:NpaNXs29SPKqhJ0U-8d7cw" pcbguid="de09cc18-a3d4-48f8-913a-f04e929a34a4" lastpulledtime="" lastsyncedchangeguid="64bdb6c9-7da9-aed6-b1db-a17abb065cc3"/>
 <plain>
 <wire x1="0" y1="39.349840625" x2="0" y2="11.43" width="0" layer="20"/>
@@
 <attribute name="VALUE" x="2.159" y="29.845" size="1.27" layer="27" ratio="10" rot="R90"/>
 </element>
-<element name="R1" library="rcl" library_urn="urn:adsk.eagle:library:334" package="R0805" package3d_urn="urn:adsk.eagle:package:23553/2" value="100" x="8.89" y="31.75" smashed="yes" rot="R90">
+<element name="R1" library="rcl" library_urn="urn:adsk.eagle:library:334" package="R0402" package3d_urn="urn:adsk.eagle:package:23547/3" value="220" x="8.89" y="31.75" smashed="yes" rot="R90">
 <attribute name="NAME" x="7.62" y="31.115" size="1.27" layer="25" rot="R90"/>
-<attribute name="POPULARITY" value="86" x="8.89" y="31.75" size="1.778" layer="27" rot="R90" display="off"/>
+<attribute name="POPULARITY" value="0" x="8.89" y="31.75" size="1.778" layer="27" rot="R90" display="off"/>
 <attribute name="SPICEPREFIX" value="R" x="8.89" y="31.75" size="1.778" layer="27" rot="R90" display="off"/>
 <attribute name="VALUE" x="11.43" y="31.115" size="1.27" layer="27" rot="R90"/>
 </element>
-<element name="R2" library="rcl" library_urn="urn:adsk.eagle:library:334" package="R0805" package3d_urn="urn:adsk.eagle:package:23553/2" value="120" x="13.97" y="31.75" smashed="yes" rot="R270">
+<element name="R2" library="rcl" library_urn="urn:adsk.eagle:library:334" package="R0402" package3d_urn="urn:adsk.eagle:package:23547/3" value="330" x="13.97" y="31.75" smashed="yes" rot="R270">
 <attribute name="NAME" x="15.24" y="32.385" size="1.27" layer="25" rot="R270"/>
-<attribute name="POPULARITY" value="86" x="13.97" y="31.75" size="1.778" layer="27" rot="R270" display="off"/>
+<attribute name="POPULARITY" value="0" x="13.97" y="31.75" size="1.778" layer="27" rot="R270" display="off"/>
 <attribute name="SPICEPREFIX" value="R" x="13.97" y="31.75" size="1.778" layer="27" rot="R270" display="off"/>
 <attribute name="VALUE" x="11.43" y="32.385" size="1.27" layer="27" rot="R270"/>
@@
 <attribute name="SPICEPREFIX" value="C" x="11.43" y="29.21" size="1.778" layer="27" rot="R270" display="off"/>
 <attribute name="VALUE" x="8.89" y="30.48" size="1.27" layer="27" rot="R270"/>
+</element>
+<element name="R3" library="rcl" library_urn="urn:adsk.eagle:library:334" package="R0402" package3d_urn="urn:adsk.eagle:package:23547/3" value="1000" x="11.43" y="34.29" smashed="yes" rot="R180">
+<attribute name="NAME" x="12.065" y="33.02" size="1.27" layer="25" rot="R180"/>
+<attribute name="POPULARITY" value="0" x="11.43" y="34.29" size="1.778" layer="27" rot="R180" display="off"/>
+<attribute name="SPICEPREFIX" value="R" x="11.43" y="34.29" size="1.778" layer="27" rot="R180" display="off"/>
+<attribute name="VALUE" x="12.065" y="36.83" size="1.27" layer="27" rot="R180"/>
 </element>
 </elements>
@@
 <contactref element="J2" pad="2"/>
 <contactref element="J2" pad="1"/>
-<wire x1="18.845" y1="31.75" x2="17.78" y2="31.75" width="0.3048" layer="1"/>
-<wire x1="17.78" y1="31.75" x2="16.51" y2="33.02" width="0.3048" layer="1"/>
-<wire x1="16.51" y1="33.02" x2="14.29" y2="33.02" width="0.3048" layer="1"/>
-<wire x1="14.29" y1="33.02" x2="13.97" y2="32.7" width="0.3048" layer="1"/>
 <contactref element="C4" pad="2"/>
 <wire x1="8.89" y1="25.72" x2="10.48" y2="25.72" width="0.3048" layer="1"/>
@@
 <wire x1="13.97" y1="25.72" x2="12.38" y2="25.72" width="0.3048" layer="1"/>
 <wire x1="12.38" y1="25.72" x2="11.43" y2="26.67" width="0.3048" layer="1"/>
-<wire x1="18.845" y1="31.75" x2="21.795" y2="31.75" width="0" layer="19" extent="1-1"/>
-<wire x1="11.43" y1="28.26" x2="13.97" y2="32.7" width="0" layer="19" extent="1-1"/>
-<wire x1="7" y1="16.58" x2="7" y2="22.18" width="0" layer="19" extent="1-1"/>
-<wire x1="7" y1="13.38" x2="7" y2="16.58" width="0" layer="19" extent="1-1"/>
-<wire x1="18.4" y1="22.18" x2="13.97" y2="25.72" width="0" layer="19" extent="1-1"/>
-<wire x1="18.4" y1="20.58" x2="18.4" y2="22.18" width="0" layer="19" extent="1-1"/>
-<wire x1="18.4" y1="16.58" x2="18.4" y2="20.58" width="0" layer="19" extent="1-1"/>
-<wire x1="18.4" y1="14.98" x2="18.4" y2="16.58" width="0" layer="19" extent="1-1"/>
-<wire x1="18.4" y1="14.18" x2="18.4" y2="14.98" width="0" layer="19" extent="1-1"/>
+<contactref element="R3" pad="1"/>
+<wire x1="11.93" y1="34.29" x2="12.7" y2="34.29" width="0.3048" layer="1"/>
+<wire x1="12.7" y1="34.29" x2="13.97" y2="33.02" width="0.3048" layer="1"/>
+<wire x1="13.97" y1="33.02" x2="13.97" y2="32.25" width="0.3048" layer="1"/>
 </signal>
 <signal name="VDD">
@@
 <wire x1="3.81" y1="33.02" x2="5.08" y2="34.29" width="0.3048" layer="1"/>
 <wire x1="5.08" y1="34.29" x2="7.3" y2="34.29" width="0.3048" layer="1"/>
-<wire x1="7.3" y1="34.29" x2="8.89" y2="32.7" width="0.3048" layer="1"/>
+<wire x1="7.3" y1="34.29" x2="8.89" y2="32.25" width="0.3048" layer="1"/>
 </signal>
 <signal name="VIN">
@@
 <contactref element="C1" pad="1"/>
 <contactref element="C2" pad="1"/>
-<wire x1="8.89" y1="27.62" x2="8.89" y2="30.8" width="0.3048" layer="1"/>
-<wire x1="13.97" y1="30.8" x2="13.97" y2="27.62" width="0.3048" layer="1"/>
+<wire x1="8.89" y1="27.62" x2="8.89" y2="31.25" width="0.3048" layer="1"/>
+<wire x1="13.97" y1="31.25" x2="13.97" y2="27.62" width="0.3048" layer="1"/>
 <wire x1="6.8048" y1="17.9848" x2="7" y2="18.18" width="0.3048" layer="1"/>
 <wire x1="13.97" y1="27.62" x2="15.56" y2="27.62" width="0.3048" layer="1"/>
@@
 <wire x1="15.64" y1="18.18" x2="7" y2="18.18" width="0.3048" layer="1"/>
 <contactref element="C4" pad="1"/>
-<wire x1="11.43" y1="30.16" x2="10.79" y2="30.8" width="0.3048" layer="1"/>
-<wire x1="10.79" y1="30.8" x2="8.89" y2="30.8" width="0.3048" layer="1"/>
-<wire x1="11.43" y1="30.16" x2="12.07" y2="30.8" width="0.3048" layer="1"/>
-<wire x1="12.07" y1="30.8" x2="13.97" y2="30.8" width="0.3048" layer="1"/>
+<contactref element="R3" pad="2"/>
+<wire x1="8.89" y1="31.25" x2="10.34" y2="31.25" width="0.3048" layer="1"/>
+<wire x1="10.34" y1="31.25" x2="11.27" y2="30.32" width="0.3048" layer="1"/>
+<wire x1="11.27" y1="30.32" x2="11.43" y2="30.16" width="0.3048" layer="1"/>
+<wire x1="13.97" y1="31.25" x2="12.2" y2="31.25" width="0.3048" layer="1"/>
+<wire x1="12.2" y1="31.25" x2="11.27" y2="30.32" width="0.3048" layer="1"/>
+<wire x1="10.93" y1="34.29" x2="10.34" y2="33.7" width="0.3048" layer="1"/>
+<wire x1="10.34" y1="33.7" x2="10.34" y2="31.25" width="0.3048" layer="1"/>
 </signal>
 <signal name="RX">

Commit message: Updated text for pcb
Parts:
- moved R2 5.08 mm to (14.0, 36.8), turned to 180 degrees
- moved C4 2.54 mm to (11.4, 26.7)
- moved R3 2.54 mm to (11.4, 36.8)
- moved C1 1.27 mm to (7.62, 26.7)
- moved C2 1.27 mm to (15.2, 26.7)
Routing:
- net GND: track 23.0 -> 15.8 mm
- net VIN: track 37.3 -> 43.9 mm
- net TX: track 15.7 -> 13.6 mm
- net RX: track 9.43 -> 7.42 mm
Other:
- board text added: "GND"
- board text added: "RX"
- board text added: "TX"
- board text added: "VDD"
